File: full.sch (EAGLE design)
At the start: 21 parts, among them X1 OPAMP

Commit message: Circuit additions
Parts:
- added C2: 500n, rcl:C-EU025-025X050
- added C3: 100u, rcl:C-EU025-025X050
- added D1: 1N4004, diode:1N4004
- added OK1: SFH618A-2, optocoupler:SFH618A-2
- added R17: 100, rcl:R-EU_0204/7
- added R18: 220, rcl:R-EU_0204/7
- added R19: 1Meg, rcl:R-EU_0204/7
- J1: value (none) -> 4x4 Keypad
Connections:
- new net 0: OK1.C
- new net N$16: J1.1, U$1.A0
- new net N$28: U$1.A5
- new net N$29: C1.2, C2.2, R17.1
- new net N$30: OK1.A, R18.2
- new net N$31: C3.2, D1.C, OK1.EMIT, R19.2
- new net VCC: OK1.COL
- net GND: now also C2.1, C3.1, D1.A, R19.1
- net N$17: now also R17.2, X1.N; no longer C1.2, X1.P
- net N$22: now also U$1.A4; no longer U$1.D13
- net N$23: now also R18.1, U$1.D13; no longer J1.4, U$1.A0
- net N$24: now also J1.2; no longer J1.3
- net N$25: now also J1.3; no longer J1.2
- net N$26: now also J1.4; no longer J1.1
- net N$8: now also X1.P; no longer X1.N
Other:
- note added: "I need to check if this work out due to the DC blocking cap at the end"
- note added: "Keypad"
- note added: "PTT"
- note removed: "Touchpad"
- moved on the sheet: C1, SP1, X1

Commit message: Full Schematic
Parts:
- added C4: 100u, rcl:C-EU025-024X044
- added C5: (no value), rcl:C-EU025-024X044
- added C6, C7: 100u, rcl:C-EU025-025X050
- added D2: 1N5817-B, diode:1N5817-B
- added J2, J3: (no value), con-jack:DCJ0303
- added Q1: (no value), ngspice-simulation:BJT_NPN
- added R20: 100, rcl:R-EU_0207/10
- added R21: 20, rcl:R-EU_0207/10
- added R22: 1k, rcl:R-EU_0207/10
- added R23: 220, rcl:R-EU_0207/10
- added R24: (no value), rcl:R-EU_0204/7
- added R25, R26: 10k, rcl:POTENTIOMETER_PT-10
Connections:
- new net N$32: C5.2, D2.C, R24.2, U$1.A5
- new net N$33: Q1.E, R21.2
- new net N$34: C4.1, Q1.B, R22.1, R23.2
- new net N$35: C4.2
- new net N$36: C7.1, J2.3
- new net N$37: J2.2
- new net N$38: C6.1, J3.2, J3.3
- new net N$39: C6.2
- new net N$40: C7.2
- new net N$41: R26.3, U$1.A7
- new net N$42: R25.3, U$1.A6
- net +5V: now also R20.2, R22.2, R25.2, R26.2
- net 0: now also C5.1, J2.1, J3.1, R21.1, R23.1, R24.1, R25.1, R26.1
- net N$28: now also D2.A, Q1.C, R20.1; no longer U$1.A5
Other:
- note added: "PC In"
- note added: "PC Out"
- note added: "Radio In"
- note added: "Radio Out"
- note added: "Right PC Out"
- note added: "VOX-Hold"
- note added: "VOX-Sensitivity"
